File: stm32mp2-core.kicad_sch (KiCad schematic)
At the start: 0 parts

Commit message: did more stuff
Other:
- note added: "ref schema"
Changed lines of the file:
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@@
 	(generator_version "9.0")
 	(paper "A4")
+	(text "ref schema"
+		(exclude_from_sim no)
+		(at 56.896 186.436 0)
+		(effects
+			(font
+				(size 10 10)
+				(thickness 2)
+				(bold yes)
+			)
+			(href "file://mb1605-mp257f-c01-schematic.pdf")
+		)
+	)
 	(sheet
 		(at 121.92 60.96)
