File: stm32mp25-pg2.kicad_sch (KiCad schematic)
At the start: 1 part, among them U1 STM32MP257FAI3

Commit message: connected lpddr4 to mp
Parts:
- U1: footprint TFBGA436_STM -> STM32MP257FAI3:TFBGA436_STM
Changed lines of the file:
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@@
 	(bus_alias "DDR"
 		(members "DQ0_[0..7]" "DQ1_[0..7]" "DQ2_[0..7]" "DQ3_[0..7]" "DQS0-" "DQS0+"
-			"DQS1-" "DQS1+" "DQS2-" "DQS2+" "DQS3-" "DQS3+" "ZQ" "A0_[0..7]" "A1_[0..7]"
-			"A2_[0..7]" "A3_[0..7]" "DQM0" "DQM1" "DQM2" "DQM3" "RESET#"
+			"DQS1-" "DQS1+" "DQS2-" "DQS2+" "DQS3-" "DQS3+" "ZQ0" "RESET#" "CAA[0..5]"
+			"CAB[0..5]" "CSA0" "CSA1" "CSB0" "CSB1" "CLKA+" "CLKA-" "CLKB+" "CLKB-"
+			"CLKEA+" "CLKEA-" "CLKEB+" "CLKEB-" "DMIA0" "DMIA1" "DMIB0" "DMIB1" "ZQ1"
 		)
 	)
@@
 			)
 		)
-		(property "Footprint" "TFBGA436_STM"
+		(property "Footprint" "STM32MP257FAI3:TFBGA436_STM"
 			(at 181.61 92.71 0)
 			(effects
