File: stm32mp25-pg3.kicad_sch (KiCad schematic)
At the start: 1 part, among them U1 STM32MP257FAI3

Commit message: did more stuff
Connections:
- net CAM.IMU_INT2: now reaches U1.A11 (PB10)
- net CAM.IMU_INT1: now reaches U1.A12 (PB9)
- net EMMC.D4: now reaches U1.A19 (PE10)
- net EMMC.CLK: now reaches U1.A20 (PE14)
- net WIFI_SDIO3.CMD: now reaches U1.A21 (PD12)
- net BT_DEV_WAKE: now reaches U1.AB4 (PB15)
- net GPIO.SAI4_SDB: now reaches U1.B11 (PB5)
- net CAM.EN: now reaches U1.B12 (PB11)
- net EMMC.D0: now reaches U1.B19 (PE13)
- net WIFI_SDIO3.D2: now reaches U1.B20 (PB12)
- net WIFI_SDIO3.D1: now reaches U1.B21 (PD13)
- net HDMI_I2S.SDO: now reaches U1.C10 (PB2)
- net HDMI.RST: now reaches U1.C12 (PB6)
- net MMC.DET: now reaches U1.C15 (PD3)
- net EMMC.D2: now reaches U1.C18 (PE8)
- net EMMC.D3: now reaches U1.C19 (PE12)
- net WIFI_SDIO3.D0: now reaches U1.C20 (PB14)
- net HDMI.INT: now reaches U1.D10 (PB4)
- net CAM.RST: now reaches U1.D11 (PB1)
- net CAM.TOF_LPn: now reaches U1.D12 (PB7)
- net GPIO.SAI4_FSA: now reaches U1.D14 (PD0)
- net EMMC.D7: now reaches U1.D17 (PE7)
- net EMMC.D5: now reaches U1.D18 (PE9)
- net WIFI_SDIO3.CLK: now reaches U1.D19 (PB13)
- net HDMI_I2S.WS: now reaches U1.E10 (PB3)
- net GPIO.SAI4_SCKA: now reaches U1.E14 (PD2)
- net GPIO.SAI4_SDA: now reaches U1.E15 (PD1)
- net EMMC.D6: now reaches U1.E16 (PE6)
- net EMMC.D1: now reaches U1.E17 (PE11)
- net I2C7.SCL: now reaches U1.F16 (PD15)
- net EMMC.CMD: now reaches U1.F17 (PE15)
- net CAM.TOF_INT: now reaches U1.G11 (PB8)
- net I2C7.SDA: now reaches U1.G15 (PD14)
- net T_PWR_EN renamed HDMI_I2S.SCK
Other:
- note added: "PMIC"

Commit message: did stuff
Connections:
- net VBUS_DIV: now reaches U1.AA6 (PF10)
- net UART6.RX: now reaches U1.H1 (PF14)
- net BT_PCM_SDI: now reaches U1.K3 (PF12)
- net UART6.TX: now reaches U1.L4 (PF13)
- net UART6.CTS: now reaches U1.L7 (PF15)
- net GPIO.SPI6_SCK: now reaches U1.T9 (PF7)
- net I2C2.SCL: now reaches U1.V10 (PF2)
- net I2C2.SDA: now reaches U1.V12 (PF0)
- net ETH1.CLK: now reaches U1.W10 (PF3)
- net ETH1.RXD0: now reaches U1.W11 (PF1)
- net GPIO.SPI6_NSS: now reaches U1.Y10 (PF4)
- net MCO1: now reaches U1.Y6 (PF11)
- net VCONN_CC1_EN: now reaches U1.Y9 (PF5)
Other:
- note added: "PERIPH"

Commit message: connected lpddr4 to mp
Parts:
- U1: footprint TFBGA436_STM -> STM32MP257FAI3:TFBGA436_STM
Changed lines of the file:
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@@
 			)
 		)
-		(property "Footprint" "TFBGA436_STM"
+		(property "Footprint" "STM32MP257FAI3:TFBGA436_STM"
 			(at 190.5 80.01 0)
 			(effects
