File: stm32mp25-pg4.kicad_sch (KiCad schematic)
At the start: 1 part, among them U1 STM32MP257FAI3

Commit message: did stuff
Connections:
- net BT_REG_ON: now reaches U1.AA4 (PG4)
- net BT_PCM_CLK: now reaches U1.H2 (PG6)
- net UART5.TX: now reaches U1.H3 (PG10)
- net UART5.RX: now reaches U1.J4 (PG11)
- net BT_PCM_WS: now reaches U1.K4 (PG7)
- net UART6.RTS: now reaches U1.L1 (PG5)
- net WL_REG_ON: now reaches U1.L5 (PG8)
- net TCPP_INT#: now reaches U1.W6 (PG1)
- net BT_HOST_WAKE: now reaches U1.Y4 (PG2)

Commit message: connected lpddr4 to mp
Parts:
- U1: footprint TFBGA436_STM -> STM32MP257FAI3:TFBGA436_STM
Changed lines of the file:
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@@
 			)
 		)
-		(property "Footprint" "TFBGA436_STM"
+		(property "Footprint" "STM32MP257FAI3:TFBGA436_STM"
 			(at 165.1 80.01 0)
 			(effects
