File: stm32mp25-pg5.kicad_sch (KiCad schematic)
At the start: 1 part, among them U1 STM32MP257FAI3

Commit message: connected lpddr4 to mp
Parts:
- U1: footprint TFBGA436_STM -> STM32MP257FAI3:TFBGA436_STM
Changed lines of the file:
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@@
 			)
 		)
-		(property "Footprint" "TFBGA436_STM"
+		(property "Footprint" "STM32MP257FAI3:TFBGA436_STM"
 			(at 43.18 81.28 0)
 			(effects
@@
 			)
 		)
-		(property "Footprint" "TFBGA436_STM"
+		(property "Footprint" "STM32MP257FAI3:TFBGA436_STM"
 			(at 186.69 85.09 0)
 			(effects
@@
 			)
 		)
-		(property "Footprint" "TFBGA436_STM"
+		(property "Footprint" "STM32MP257FAI3:TFBGA436_STM"
 			(at 327.66 109.22 0)
 			(effects
